File: badger-2040-wlan.kicad/badger-2040-wlan.kicad_sch (KiCad schematic)
At the start: 6 parts, among them U1 Badger2040_Conn, U3 SN74LVC1G14DBV, U4 ESP_01S_Breakout, U5 PCF8523_RTC_Breakouut

Commit message: Rev 4: removed pullup and inverter for RTC (INT_SQW)
Parts:
- removed R1: 100K, Resistor_SMD:R_0402_1005Metric, symbol Device:R
- removed U3: SN74LVC1G14DBV, Package_TO_SOT_SMD:SOT-23-5, symbol 74xGxx:SN74LVC1G14DBV
- U1: footprint user:PinSocket_1x11_P2.54mm_Horizontal_Back -> user:PinSocket_1x10_P2.54mm_Horizontal_Back
- U5: value PCF8523_RTC_Breakouut -> PCF8523_RTC_Breakout; symbol user:PCF8523_RTC_Breakouut -> user:PCF8523_RTC_Breakout
Changed lines of the file:
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@@
   (title_block
     (title "badger-240-wlan")
-    (date "2022-10-22")
-    (rev "3")
+    (date "2022-11-12")
+    (rev "4")
     (company "Bernhard Bablok")
     (comment 1 "https://github.com/bablokb/pcb-badger2040-wlan")
   )
-  (junction (at 141.605 90.17) (diameter 0) (color 0 0 0 0)
-  )
   (junction (at 97.155 103.505) (diameter 0) (color 0 0 0 0)
   )
   (junction (at 97.155 90.17) (diameter 0) (color 0 0 0 0)
   )
-  (junction (at 136.525 127) (diameter 0) (color 0 0 0 0)
-  )
-  (junction (at 149.86 113.665) (diameter 0) (color 0 0 0 0)
-  )
   (junction (at 117.475 74.93) (diameter 0) (color 0 0 0 0)
   )
-  (junction (at 131.445 67.31) (diameter 0) (color 0 0 0 0)
-  )
   (junction (at 120.65 67.31) (diameter 0) (color 0 0 0 0)
   )
@@
   )
   (junction (at 123.825 67.31) (diameter 0) (color 0 0 0 0)
-  )
-  (junction (at 149.86 127) (diameter 0) (color 0 0 0 0)
   )
   (no_connect (at 97.155 114.3))
@@
     (stroke (width 0) (type default) (color 0 0 0 0))
   )
-  (wire (pts (xy 141.605 90.17) (xy 141.605 114.3))
-    (stroke (width 0) (type default) (color 0 0 0 0))
-  )
-  (wire (pts (xy 167.64 131.445) (xy 162.56 131.445))
-    (stroke (width 0) (type default) (color 0 0 0 0))
-  )
   (wire (pts (xy 92.71 77.47) (xy 97.155 77.47))
     (stroke (width 0) (type default) (color 0 0 0 0))
@@
     (stroke (width 0) (type default) (color 0 0 0 0))
   )
-  (wire (pts (xy 131.445 67.31) (xy 149.86 67.31))
-    (stroke (width 0) (type default) (color 0 0 0 0))
-  )
   (wire (pts (xy 120.65 119.38) (xy 120.65 67.31))
     (stroke (width 0) (type default) (color 0 0 0 0))
@@
     (stroke (width 0) (type default) (color 0 0 0 0))
   )
-  (wire (pts (xy 167.64 113.665) (xy 167.64 131.445))
-    (stroke (width 0) (type default) (color 0 0 0 0))
-  )
-  (wire (pts (xy 141.605 90.17) (xy 147.955 90.17))
-    (stroke (width 0) (type default) (color 0 0 0 0))
-  )
-  (wire (pts (xy 97.155 90.17) (xy 141.605 90.17))
+  (wire (pts (xy 97.155 90.17) (xy 147.955 90.17))
     (stroke (width 0) (type default) (color 0 0 0 0))
   )
@@
     (stroke (width 0) (type default) (color 0 0 0 0))
   )
-  (wire (pts (xy 149.86 127) (xy 149.86 131.445))
-    (stroke (width 0) (type default) (color 0 0 0 0))
-  )
   (wire (pts (xy 97.155 90.17) (xy 97.155 103.505))
     (stroke (width 0) (type default) (color 0 0 0 0))
   )
-  (wire (pts (xy 149.86 131.445) (xy 154.94 131.445))
-    (stroke (width 0) (type default) (color 0 0 0 0))
-  )
-  (wire (pts (xy 149.86 113.665) (xy 149.86 67.31))
-    (stroke (width 0) (type default) (color 0 0 0 0))
-  )
   (wire (pts (xy 147.955 119.38) (xy 147.955 90.17))
     (stroke (width 0) (type default) (color 0 0 0 0))
   )
-  (wire (pts (xy 149.86 116.84) (xy 149.86 113.665))
+  (wire (pts (xy 149.86 67.31) (xy 149.86 116.84))
     (stroke (width 0) (type default) (color 0 0 0 0))
   )
@@
     (stroke (width 0) (type default) (color 0 0 0 0))
   )
-  (wire (pts (xy 151.765 127) (xy 149.86 127))
+  (wire (pts (xy 126.365 127) (xy 151.765 127))
     (stroke (width 0) (type default) (color 0 0 0 0))
   )
@@
     (stroke (width 0) (type default) (color 0 0 0 0))
   )
-  (wire (pts (xy 136.525 127) (xy 126.365 127))
-    (stroke (width 0) (type default) (color 0 0 0 0))
-  )
   (wire (pts (xy 142.875 124.46) (xy 142.875 69.85))
     (stroke (width 0) (type default) (color 0 0 0 0))
@@
     (stroke (width 0) (type default) (color 0 0 0 0))
   )
-  (wire (pts (xy 136.525 92.71) (xy 136.525 106.68))
-    (stroke (width 0) (type default) (color 0 0 0 0))
-  )
   (wire (pts (xy 126.365 74.93) (xy 126.365 108.585))
     (stroke (width 0) (type default) (color 0 0 0 0))
   )
-  (wire (pts (xy 92.71 92.71) (xy 136.525 92.71))
-    (stroke (width 0) (type default) (color 0 0 0 0))
-  )
   (wire (pts (xy 126.365 127) (xy 126.365 118.745))
     (stroke (width 0) (type default) (color 0 0 0 0))
   )
-  (wire (pts (xy 149.86 113.665) (xy 167.64 113.665))
-    (stroke (width 0) (type default) (color 0 0 0 0))
-  )
   (wire (pts (xy 114.935 119.38) (xy 120.65 119.38))
     (stroke (width 0) (type default) (color 0 0 0 0))
@@
     (stroke (width 0) (type default) (color 0 0 0 0))
   )
-  (wire (pts (xy 131.445 67.31) (xy 131.445 114.3))
-    (stroke (width 0) (type default) (color 0 0 0 0))
-  )
   (wire (pts (xy 97.155 103.505) (xy 97.155 111.76))
     (stroke (width 0) (type default) (color 0 0 0 0))
@@
     (stroke (width 0) (type default) (color 0 0 0 0))
   )
-  (wire (pts (xy 136.525 127) (xy 136.525 119.38))
-    (stroke (width 0) (type default) (color 0 0 0 0))
-  )
   (wire (pts (xy 117.475 74.93) (xy 126.365 74.93))
     (stroke (width 0) (type default) (color 0 0 0 0))
   )
-  (wire (pts (xy 123.825 67.31) (xy 131.445 67.31))
-    (stroke (width 0) (type default) (color 0 0 0 0))
-  )
-  (wire (pts (xy 149.86 127) (xy 136.525 127))
+  (wire (pts (xy 123.825 67.31) (xy 149.86 67.31))
     (stroke (width 0) (type default) (color 0 0 0 0))
   )
@@
     (property "Reference" "U1" (id 0) (at 85.09 60.325 0))
     (property "Value" "Badger2040_Conn" (id 1) (at 85.09 63.5 0))
-    (property "Footprint" "user:PinSocket_1x11_P2.54mm_Horizontal_Back" (id 2) (at 90.17 71.12 0)
+    (property "Footprint" "user:PinSocket_1x10_P2.54mm_Horizontal_Back" (id 2) (at 90.17 71.12 0)
       (effects (font (size 1.27 1.27)) hide)
     )
@@
     (pin "1")
     (pin "10")
-    (pin "11")
     (pin "2")
     (pin "3")
@@
     (pin "9")
   )
-  (symbol (lib_id "74xGxx:SN74LVC1G14DBV") (at 136.525 114.3 90) (unit 1)
-    (in_bom yes) (on_board yes)
-    (property "Reference" "U3" (id 0) (at 136.525 130.175 90))
-    (property "Value" "SN74LVC1G14DBV" (id 1) (at 136.525 132.715 90))
-    (property "Footprint" "Package_TO_SOT_SMD:SOT-23-5" (id 2) (at 142.875 114.3 0)
-      (effects (font (size 1.27 1.27)) hide)
-    )
-    (property "Datasheet" "http://www.ti.com/lit/ds/symlink/sn74lvc1g14.pdf" (id 3) (at 136.525 114.3 0)
-      (effects (font (size 1.27 1.27)) hide)
-    )
-    (property "LCSC" "C434069" (id 4) (at 136.525 114.3 0)
-      (effects (font (size 1.27 1.27)) hide)
-    )
-    (pin "1")
-    (pin "2")
-    (pin "3")
-    (pin "4")
-    (pin "5")
-  )
-  (symbol (lib_id "Device:R") (at 158.75 131.445 90) (unit 1)
-    (in_bom yes) (on_board yes)
-    (property "Reference" "R1" (id 0) (at 158.75 134.62 90))
-    (property "Value" "100K" (id 1) (at 158.75 131.445 90))
-    (property "Footprint" "Resistor_SMD:R_0402_1005Metric" (id 2) (at 158.75 133.223 90)
-      (effects (font (size 1.27 1.27)) hide)
-    )
-    (property "Datasheet" "~" (id 3) (at 158.75 131.445 0)
-      (effects (font (size 1.27 1.27)) hide)
-    )
-    (property "LCSC" "C25741" (id 4) (at 158.75 131.445 0)
-      (effects (font (size 1.27 1.27)) hide)
-    )
-    (pin "1")
-    (pin "2")
-  )
   (symbol (lib_id "power:+3V3") (at 123.825 67.31 0) (unit 1)
     (in_bom yes) (on_board yes) (fields_autoplaced)
@@
     (pin "2")
   )
-  (symbol (lib_id "user:PCF8523_RTC_Breakouut") (at 155.575 119.38 0) (unit 1)
+  (symbol (lib_id "user:PCF8523_RTC_Breakout") (at 155.575 119.38 0) (unit 1)
     (in_bom no) (on_board yes)
-    (property "Reference" "U5" (id 0) (at 158.75 107.315 0)
+    (property "Reference" "U5" (id 0) (at 157.48 109.22 0)
       (effects (font (size 1.27 1.27)) (justify left))
     )
-    (property "Value" "PCF8523_RTC_Breakouut" (id 1) (at 153.035 110.49 0)
+    (property "Value" "PCF8523_RTC_Breakout" (id 1) (at 152.4 112.395 0)
       (effects (font (size 1.27 1.27)) (justify left))
     )
-    (property "Footprint" "user:PCF8523_Breakout" (id 2) (at 155.575 119.38 0)
+    (property "Footprint" "user:PCF8523_Breakout" (id 2) (at 158.115 130.81 0)
       (effects (font (size 1.27 1.27)) hide)
     )
@@
       (reference "JP1") (unit 1) (value "Jumper_2_Open") (footprint "Jumper:SolderJumper-2_P1.3mm_Open_Pad1.0x1.5mm")
     )
-    (path "/7b06f186-f0c9-4b2b-9d8f-7fde4d5b7001"
-      (reference "R1") (unit 1) (value "100K") (footprint "Resistor_SMD:R_0402_1005Metric")
-    )
     (path "/2bc26db0-e59c-43b0-976d-4f9e2b8c27ff"
-      (reference "U1") (unit 1) (value "Badger2040_Conn") (footprint "user:PinSocket_1x11_P2.54mm_Horizontal_Back")
-    )
-    (path "/74340138-d72a-4ff3-9cdb-c74565e3610c"
-      (reference "U3") (unit 1) (value "SN74LVC1G14DBV") (footprint "Package_TO_SOT_SMD:SOT-23-5")
+      (reference "U1") (unit 1) (value "Badger2040_Conn") (footprint "user:PinSocket_1x10_P2.54mm_Horizontal_Back")
     )
     (path "/adb2dcb9-f310-47fc-a32d-61fdb74a70e8"
@@
     )
     (path "/aabe08f7-a1b1-4704-8e83-d37349a2b92f"
-      (reference "U5") (unit 1) (value "PCF8523_RTC_Breakouut") (footprint "user:PCF8523_Breakout")
-    )
-  )
+      (reference "U5") (unit 1) (value "PCF8523_RTC_Breakout") (footprint "user:PCF8523_Breakout")
+    )
+  )
